Commit message: Camera added

File: urdf/baxter.urdf.xacro (robot description, xacro)
@@ -3,4 +3,5 @@
   <xacro:arg name="gazebo" default="false"/>
   <xacro:arg name="pedestal" default="true"/>
+  <xacro:include filename="$(find baxter_description)/urdf/common.xacro" />
   <!-- Baxter Base URDF -->
   <xacro:include filename="$(find baxter_description)/urdf/baxter_base/baxter_base.urdf.xacro">
@@ -20,5 +21,5 @@
     <xacro:include filename="$(find baxter_description)/urdf/sensors/kinect2.urdf.xacro" />
     <xacro:kinect2_v0 name="head_mount" parent="base" >
-      <origin xyz="0.2 0 0.091746" rpy="0 0 0" />
+      <origin xyz="0 0 0.45" rpy="0 0.9 0" />
     </xacro:kinect2_v0>
 </robot>

File: urdf/sensors/kinect2.urdf.xacro (robot description, xacro)
@@ -34,8 +34,45 @@
       </collision>
     </link>
+    <!-- kinect2 ir sensor physical attachment -->
+    <joint name="${name}_kinect2_ir_joint" type="fixed">
+      <origin xyz="-0.032267 -0.0475 0.155" rpy="0 0 0"/>
+      <parent link="${name}_kinect2_link"/>
+      <child link="${name}_kinect2_ir_link"/>
+    </joint>
+    <link name="${name}_kinect2_ir_link">
+      <inertial>
+        <mass value="0.1" />
+        <origin xyz="0 0 0" rpy="0 0 0"/>
+        <inertia ixx="0.01"  ixy="0.0"  ixz="0.0"
+                 iyy="0.01"  iyz="0.0"
+                 izz="0.01" />
+      </inertial>
+      <visual>
+        <origin xyz="0.0 0.0 0" rpy="0 0 0"/>
+        <geometry>
+          <sphere radius="0.0005"/>
+        </geometry>
+      </visual>
+      <collision>
+        <origin xyz="0.0 0.0 0" rpy="0 0 0"/>
+        <geometry>
+          <sphere radius="0.0005"/>
+        </geometry>
+      </collision>
+    </link>
+    <!-- kinect2 ir sensor frame -->
+    <joint name="${name}_kinect2_ir_optical_frame_joint" type="fixed">
+      <origin xyz="${cal_kinect_x}                  ${cal_kinect_y+ir_depth_rgb_offset_y} ${cal_kinect_z}"
+              rpy="${-M_PI/2+cal_kinect_roll}       ${0.0+cal_kinect_pitch}               ${-M_PI/2+cal_kinect_yaw}" />
+      <parent link="${name}_kinect2_ir_link"/>
+      <child link="${name}_kinect2_ir_optical_frame"/>
+    </joint>
+    <link name="${name}_kinect2_ir_optical_frame"/>
+    <!-- gazebo extensions -->
+    <xacro:kinect2_ir_gazebo_v0 link_name="${name}_kinect2_ir_link" frame_name="${name}_kinect2_ir_optical_frame" camera_name="head_mount_kinect2" />
     <!-- kinect2 rgb sensor physical attachment -->
     <joint name="${name}_kinect2_rgb_joint" type="fixed">
       <origin xyz="0 -0.05175 0" rpy="0 0 0"/>
-      <parent link="${name}_kinect2_link"/>
+      <parent link="${name}_kinect2_ir_link"/>
       <child link="${name}_kinect2_rgb_link"/>
     </joint>
@@ -49,6 +86,6 @@
       </inertial>
       <visual>
-        <origin xyz="0 0 0"
-                rpy="0 0 0" />
+        <origin xyz="${cal_kinect_x}            ${cal_kinect_y}                 ${cal_kinect_z}"
+                rpy="${-M_PI/2+cal_kinect_roll} ${0.0+cal_kinect_pitch}         ${-M_PI/2+cal_kinect_yaw}" />
         <geometry>
           <sphere radius="0.0005"/>
@@ -64,6 +101,6 @@
     <!-- kinect2 rgb sensor frame -->
     <joint name="${name}_kinect2_rgb_optical_frame_joint" type="fixed">
-      <origin xyz="0 0 0"
-              rpy="0 0 0" />
+      <origin xyz="${cal_kinect_x}            ${cal_kinect_y}                 ${cal_kinect_z}"
+              rpy="${-M_PI/2+cal_kinect_roll} ${0.0+cal_kinect_pitch}         ${-M_PI/2+cal_kinect_yaw}" />
       <parent link="${name}_kinect2_rgb_link"/>
       <child link="${name}_kinect2_rgb_optical_frame"/>

Commit message: Camera position fixed

File: urdf/baxter.urdf.xacro (robot description, xacro)
@@ -21,5 +21,5 @@
     <xacro:include filename="$(find baxter_description)/urdf/sensors/kinect2.urdf.xacro" />
     <xacro:kinect2_v0 name="head_mount" parent="base" >
-      <origin xyz="0 0 0.45" rpy="0 0.9 0" />
+      <origin xyz="0.05 0 0.45" rpy="0 0.9 0" />
     </xacro:kinect2_v0>
 </robot>
